Commit message: update

File: usv_sim/xacro/sailboat.xacro (robot description, xacro)
@@ -34,5 +34,5 @@
 		<dynamics damping="1.0"/>
 		<axis xyz="0 0 1"/>
-		<limit effort="100" velocity="70" lower="-${PI}" upper="${PI}" />
+		<limit effort="100" velocity="70" lower="-${PI*0.5}" upper="${PI*0.5}" />
 	</joint>
 	<link name="keel">
